File: rev_b/USBCKeychainAccessory.kicad_pcb (KiCad board)
At the start: 2 copper layers, 25.4 x 39.9 mm, 67 parts, among them J1 Conn_01x10, J2 Conn_01x10, J3 Conn_01x04, P1 U261-241N-4BS60, SW1 KMS233G LFG, SW2 KMS233G LFG, U1 AP2112K-3.3, U2 RP2350_60QFN, U3 W25Q32JVUUIQ, Y1 ABM8-272-T3

Commit message: Revision B
Parts:
- removed U1: AP2112K-3.3, Package_TO_SOT_SMD:SOT-23-5
- added U4: AMS1117-3.3V, Package_TO_SOT_SMD:SOT-89-3, F.Cu at (110.4, 47.6)
- C2, C3: footprint Capacitor_SMD:C_0402_1005Metric -> Parts:C_0402_1005Metric_small_pads
- L1: footprint Inductor_SMD:L_0603_1608Metric -> Parts:L_pol_2016
- SW1, SW2: value KMS233G LFG -> KMS221GLFS
- moved D1 9.39 mm to (105.7, 47.2), turned to 90 degrees
- moved C2 7.54 mm to (106.7, 55.2), turned to 180 degrees
- moved L1 7.24 mm to (106.7, 52.7), turned to 0 degrees
- moved R8 6.30 mm to (102.8, 45.6)
- moved C3 6.27 mm to (106.7, 54.2), turned to 180 degrees
- moved C5 5.65 mm to (98.3, 66.8)
- moved Y1 5.51 mm to (98.4, 64.4)
- moved C10 5.51 mm to (104.9, 66.5)
- moved C11 5.51 mm to (102.1, 53.2)
- moved C12 5.51 mm to (111.3, 58.1)
- moved C13 5.51 mm to (98.1, 61.1)
- moved C14 5.51 mm to (111.3, 62.0)
- moved C15 5.51 mm to (108.2, 65.0)
- moved C16 5.51 mm to (102.9, 66.5)
- moved C17 5.51 mm to (103.2, 53.2)
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Connections:
- net Net-(U2-VREG_LX) renamed /VREG_LX
- H1 pad 1: (no net) -> GND
Routing:
- net +3V3: track 90.3 -> 111.5 mm, vias 4 -> 6
- net +1V1: track 31.9 -> 24.5 mm, vias 9 -> 8
- net /VREG_LX: track 4.50 -> 0.00 mm
- net VBUS: track 23.0 -> 27.5 mm
- net Net-(U2-USB_DM): track 2.80 -> 6.13 mm
- net Net-(U2-USB_DP): track 3.05 -> 6.05 mm
- net +5V: track 11.2 -> 13.7 mm, vias 0 -> 1
- net /D+: track 47.0 -> 45.7 mm
- net Net-(U2-VREG_AVDD): track 4.52 -> 5.56 mm
- net /GPIO25: track 22.8 -> 21.9 mm
- net Net-(P1-CC): track 1.65 -> 2.43 mm
- net GND: vias 9 -> 15
- added copper zone on F.Cu, net /VREG_LX
Other:
- board text added: "(c) schmitworks 2025"
- board text added: "DAEDALUS PROTOTYPE REVISION B"
- board text added: "DO NOT REDISTRIBUTE"
