File: rev_b/USBCKeychainAccessory.kicad_sch (KiCad schematic)
At the start: 67 parts, among them J1 Conn_01x10, J2 Conn_01x10, J3 Conn_01x04, P1 U261-241N-4BS60, SW1 KMS233G LFG, SW2 KMS233G LFG, U1 AP2112K-3.3, U2 RP2350_60QFN, U3 W25Q32JVUUIQ, Y1 ABM8-272-T3

Commit message: Revision B
Parts:
- removed U1: AP2112K-3.3, Package_TO_SOT_SMD:SOT-23-5, symbol Regulator_Linear:AP2112K-3.3
- added U4: AMS1117-3.3V, Package_TO_SOT_SMD:SOT-89-3, symbol Regulator_Linear:AMS1117-3.3
- C2, C3: footprint Capacitor_SMD:C_0402_1005Metric -> Parts:C_0402_1005Metric_small_pads
- L1: footprint Inductor_SMD:L_0603_1608Metric -> Parts:L_pol_2016
- SW1, SW2: value KMS233G LFG -> KMS221GLFS
Connections:
- net +3V3: now also U4.2 (VO)
- net +5V: now also U4.3 (VI)
- net GND: now also H1.1 (MP), U4.1 (GND); no longer H1.MP
- net VREG_LX: now reaches L1.2, U2.48 (VREG_LX)
Other:
- note added: "* 4 MB"
- note added: "* MCU"
- note added: "* MSKSemi, SOT-89 package"
- note removed: "* 16 MB"
- moved on the sheet: C1, C10, C11, C12, C13, C14, C15, C16, C17, C18, C19, C2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
